File: Schematics/APCSboard/APCSboard.sch (KiCad schematic (older format))
At the start: 51 parts, among them J1 LOAD1_CONNECTION, J2 LOAD2_CONNECTION, J3 BOOT, J4 SENS1_CONNECTION, J5 SENS2_CONNECTION, J6 ADDSENS_CONNECTION, J7 DIO_CLK(RX)_TX, Q1 IRF40DM229, Q2 IRF40DM229, Q3 IRF40DM229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

Commit message: added 3 part
Parts:
- gave numbers to parts that had none: 2
Changed lines of the file:
@@
 $Descr A3 16535 11693
 encoding utf-8
-Sheet 1 1
+Sheet 1 2
 Title "APCSystem"
 Date "2020-03-02"
@@
 	500  7800 16050 7800
 $Comp
-L Device:Rotary_Encoder_Switch SW?
+L Device:Rotary_Encoder_Switch SW1
 U 1 1 5F111349
 P 7400 9400
-F 0 "SW?" H 7400 9767 50  0000 C CNN
+F 0 "SW1" H 7400 9767 50  0000 C CNN
 F 1 "Rotary_Encoder_Switch" H 7400 9676 50  0000 C CNN
 F 2 "" H 7250 9560 50  0001 C CNN
@@
 $EndComp
 $Comp
-L Device:R R?
+L Device:R R16
 U 1 1 5F11A8B2
 P 8150 9100
-F 0 "R?" H 8220 9146 50  0000 L CNN
+F 0 "R16" H 8220 9146 50  0000 L CNN
 F 1 "1k" H 8220 9055 50  0000 L CNN
 F 2 "" V 8080 9100 50  0001 C CNN
@@
 	8150 9300 8150 9250
 $Comp
-L power:GND #PWR?
+L power:GND #PWR040
 U 1 1 5F12546D
 P 7700 9650
-F 0 "#PWR?" H 7700 9400 50  0001 C CNN
+F 0 "#PWR040" H 7700 9400 50  0001 C CNN
 F 1 "GND" V 7705 9522 50  0000 R CNN
 F 2 "" H 7700 9650 50  0001 C CNN
@@
 	10900 4800 11950 4800
 $Comp
-L power:GND #PWR?
+L power:GND #PWR042
 U 1 1 5F1490F9
 P 11800 3500
-F 0 "#PWR?" H 11800 3250 50  0001 C CNN
+F 0 "#PWR042" H 11800 3250 50  0001 C CNN
 F 1 "GND" H 11900 3350 50  0000 R CNN
 F 2 "" H 11800 3500 50  0001 C CNN
@@
 	11800 3500 12000 3500
 $Comp
-L power:+3.3V #PWR?
+L power:+3.3V #PWR041
 U 1 1 5F1611B6
 P 8150 8750
-F 0 "#PWR?" H 8150 8600 50  0001 C CNN
+F 0 "#PWR041" H 8150 8600 50  0001 C CNN
 F 1 "+3.3V" H 8165 8923 50  0000 C CNN
 F 2 "" H 8150 8750 50  0001 C CNN
@@
 Text Notes 9700 11150 0    50   ~ 0
 ENCODER
+$Sheet
+S 14100 9400 750  150
+U 5EDBE888
+F0 "LightSensor" 50
+F1 "LightSensor.sch" 50
+$EndSheet
 $EndSCHEMATC
